Commit message: Fixed URDF, and tuned motor controllers for forbal5.

File: forbal_description/urdf/forbal5.ros2_control.xacro (robot description, xacro)
@@ -18,5 +18,5 @@
       <state_interface name="velocity"/>
       <state_interface name="effort"/>
-      <param name="Position_P_Gain">500</param>
+      <param name="Position_P_Gain">1200</param>
       <param name="Position_D_Gain">2000</param>
       <!-- <param name="Position_P_Gain">2500</param> -->
@@ -35,6 +35,6 @@
       <state_interface name="velocity"/>
       <state_interface name="effort"/>
-      <param name="Position_P_Gain">6000</param>
-      <param name="Position_D_Gain">10000</param>
+      <param name="Position_P_Gain">7000</param>
+      <param name="Position_D_Gain">12000</param>
       <!-- <param name="Position_P_Gain">12500</param> -->
       <!-- <param name="Position_D_Gain">16000</param> -->
@@ -52,8 +52,8 @@
       <state_interface name="velocity"/>
       <state_interface name="effort"/>
-      <param name="Position_P_Gain">6000</param>
-      <param name="Position_D_Gain">10000</param>
-      <param name="Position_P_Gain">14000</param>
-      <param name="Position_D_Gain">16000</param>
+      <param name="Position_P_Gain">8000</param>
+      <param name="Position_D_Gain">12000</param>
+      <!-- <param name="Position_P_Gain">14000</param> -->
+      <!-- <param name="Position_D_Gain">16000</param> -->
       <param name="Position_I_Gain">0</param>
       <param name="Velocity_P_Gain">1920</param>
@@ -69,5 +69,5 @@
       <state_interface name="velocity"/>
       <state_interface name="effort"/>
-      <param name="Position_P_Gain">1250</param>
+      <param name="Position_P_Gain">2000</param>
       <param name="Position_D_Gain">4000</param>
       <param name="Position_I_Gain">0</param>
@@ -84,5 +84,5 @@
       <state_interface name="velocity"/>
       <state_interface name="effort"/>
-      <param name="Position_P_Gain">1250</param>
+      <param name="Position_P_Gain">2000</param>
       <param name="Position_D_Gain">4000</param>
       <param name="Position_I_Gain">0</param>

File: forbal_description/urdf/forbal5.xacro (robot description, xacro)
@@ -229,5 +229,5 @@
         <parent link="ee"/>
         <child link="ee_motor"/>
-        <origin rpy="1.5707963268 0.0 0.0" xyz="0.025 -0.02100000 0.0"/>
+        <origin rpy="1.5707963268 -1.57079633 0.0" xyz="0.025 -0.02100000 0.0"/>
         <axis xyz="0.0 0.00000000 1.00000000"/>
         <limit lower="-3.14159265" upper="3.14159265" effort="0" velocity="0"/>
@@ -237,5 +237,5 @@
         <child link="ee_imp"/>
         <origin rpy="0.0 -1.5707963268  0.00000000" xyz="0.019 -0.024 -0.019"/>
-        <axis xyz="0.00000000 0.00000000 1.00000000"/>
+        <axis xyz="0.00000000 0.00000000 -1.00000000"/>
         <limit lower="-3.14159265" upper="3.14159265" effort="0" velocity="0"/>
     </joint>
