Commit message: Got injection of dummy parameter working, it is now the sim parameter in both launch fles.

File: forbal_description/urdf/forbal2.urdf.xacro (robot description, xacro)
@@ -1,7 +1,7 @@
 <?xml version="1.0"?>
 <robot name="forbal2" xmlns:xacro="http://ros.org/wiki/xacro">
-  <xacro:arg name="dummy" default="false"/>
   <xacro:include filename="$(find forbal_description)/urdf/forbal2.xacro" />
   <xacro:include filename="$(find forbal_description)/urdf/forbal2.ros2_control.xacro" />
+  <xacro:arg name="dummy" default="false"/>
   <link name="world"/>
   <xacro:forbal2 parent="world">

File: forbal_description/urdf/forbal5.urdf.xacro (robot description, xacro)
@@ -4,9 +4,10 @@
   <xacro:include filename="$(find forbal_description)/urdf/forbal2.xacro" />
   <xacro:include filename="$(find forbal_description)/urdf/forbal5.ros2_control.xacro" />
+  <xacro:arg name="dummy" default="false"/>
   <link name="world"/>
   <xacro:forbal5 parent="world">
     <origin xyz="0 0 0" rpy="0 0 0" />
   </xacro:forbal5>
-  <xacro:forbal5_ros2_control name="forbal5" dummy="false"/>
+  <xacro:forbal5_ros2_control name="forbal5" dummy="$(arg dummy)"/>
   <xacro:ringmass parent="link11" mass="0.02982881" density="8050.0" radius_inner="0.0032" radius_outer="0.02">
     <origin xyz="-0.2 0 0" rpy="0 0 0"/>

File: forbal_description/urdf/forbal5.xacro (robot description, xacro)
@@ -231,5 +231,5 @@
         <origin rpy="1.5707963268 -1.57079633 0.0" xyz="0.025 -0.02100000 0.0"/>
         <axis xyz="0.0 0.00000000 1.00000000"/>
-        <limit lower="-3.14159265" upper="3.14159265" effort="0" velocity="0"/>
+        <limit lower="-2.0" upper="1.55" effort="0" velocity="0"/>
     </joint>
     <joint name="joint4" type="revolute">
