Commit message: IK algorithm working.

File: forbal_description/urdf/forbal2.xacro (robot description, xacro)
@@ -152,19 +152,7 @@
         <parent link="ee"/>
         <child link="ee_mkr"/>
-        <origin rpy="0.00000000 0.00000000 0.00000000" xyz="0.02500000 0.00000000 0.00000000"/>
+        <origin rpy="0.00000000 0.00000000 0.00000000" xyz="0.000000 0.00000000 0.00000000"/>
         <axis xyz="100"/>
     </joint>
-    <!-- <joint name="joint_lc1_l12" type="fixed">
-        <parent link="link12"/>
-        <child link="lc1"/>
-        <origin rpy="0.00000000 0.00000000 0.00000000" xyz="0.20000000 0.04520000 0.00000000"/>
-        <axis xyz="100"/>
-    </joint>
-    <joint name="joint_lc_l22" type="fixed">
-        <parent link="link22"/>
-        <child link="lc2"/>
-        <origin rpy="0.00000000 0.00000000 0.00000000" xyz="0.20000000 -0.04100000  0.00000000"/>
-        <axis xyz="100"/>
-    </joint> -->
 </xacro:macro>
 <xacro:macro name="ringmass" params="parent mass density radius_inner radius_outer *origin ">

File: forbal_description/urdf/forbal5.xacro (robot description, xacro)
@@ -229,5 +229,5 @@
         <parent link="ee"/>
         <child link="ee_motor"/>
-        <origin rpy="1.5707963268 -1.57079633 0.0" xyz="0.025 -0.02100000 0.0"/>
+        <origin rpy="1.5707963268 -1.57079633 0.0" xyz="0.025 -0.01900000 0.0"/>
         <axis xyz="0.0 0.00000000 1.00000000"/>
         <limit lower="-2.0" upper="1.55" effort="0" velocity="0"/>
