Commit message: Added joint limits check for forbal5.

File: forbal_description/urdf/forbal5.xacro (robot description, xacro)
@@ -186,5 +186,5 @@
         <origin rpy="0.00000000 0.00000000 0.00000000" xyz="0.00000000 -0.04310000  0.22750000"/>
         <axis xyz="0.00000000 1.00000000 0.00000000"/>
-        <limit lower="-3.14159265" upper="3.14159265" effort="0" velocity="0"/>
+        <limit lower="-1.25" upper="1.45" effort="30.0" velocity="0"/>
     </joint>
     <joint name="joint12" type="revolute">
@@ -193,5 +193,5 @@
         <origin rpy="0.00000000 0.00000000 0.00000000" xyz="0.20000000 0.00000000 0.00000000"/>
         <axis xyz="0.00000000 -1.00000000  0.00000000"/>
-        <limit lower="-3.14159265" upper="3.14159265" effort="0" velocity="0"/>
+        <limit lower="-2.9" upper="2.9" effort="30.0" velocity="0"/>
     </joint>
     <joint name="joint21" type="revolute">
@@ -200,5 +200,5 @@
         <origin rpy="0.00000000 0.00000000 0.00000000" xyz="0.00000000 0.04310000 0.22750000"/>
         <axis xyz="0.00000000 -1.00000000  0.00000000"/>
-        <limit lower="-3.14159265" upper="3.14159265" effort="0" velocity="0"/>
+        <limit lower="-1.5" upper="1.25" effort="30.0" velocity="0"/>
     </joint>
     <joint name="joint22" type="revolute">
@@ -207,5 +207,5 @@
         <origin rpy="0.00000000 0.00000000 0.00000000" xyz="0.20000000 0.00000000 0.00000000"/>
         <axis xyz="0.00000000 1.00000000 0.00000000"/>
-        <limit lower="-3.14159265" upper="3.14159265" effort="0" velocity="0"/>
+        <limit lower="0.3" upper="2.9" effort="30.0" velocity="0"/>
     </joint>
     <joint name="joint_lc1_l12" type="fixed">

Commit message: Circle trajectories generated.

File: forbal_description/urdf/forbal5.xacro (robot description, xacro)
@@ -186,5 +186,5 @@
         <origin rpy="0.00000000 0.00000000 0.00000000" xyz="0.00000000 -0.04310000  0.22750000"/>
         <axis xyz="0.00000000 1.00000000 0.00000000"/>
-        <limit lower="-1.25" upper="1.45" effort="30.0" velocity="0"/>
+        <limit lower="-1.27" upper="1.45" effort="30.0" velocity="0"/>
     </joint>
     <joint name="joint12" type="revolute">
@@ -243,5 +243,5 @@
         <parent link="ee_imp"/>
         <child link="ee_mkr"/>
-        <origin rpy="3.1415926536 0.0 -1.5707963268" xyz="0.0 -0.02 -0.01"/>
+        <origin rpy="3.1415926536 0.0 -1.5707963268" xyz="0.0 0.0 0.0"/>
     </joint>
 </xacro:macro>
