Commit message: configured joint state correction for rviz, some error in joints, still working out.

File: forbal_description/urdf/forbal2.ros2_control.xacro (robot description, xacro)
@@ -1,5 +1,5 @@
 <?xml version="1.0"?>
 <robot xmlns:xacro="http://www.ros.org/wiki/xacro">
-  <xacro:macro name="forbal_ros2_control" params="name dummy">
+  <xacro:macro name="forbal2_ros2_control" params="name dummy">
     <ros2_control name="${name}" type="system">
       <hardware>

File: forbal_description/urdf/forbal2.urdf.xacro (robot description, xacro)
@@ -1,4 +1,5 @@
 <?xml version="1.0"?>
-<robot name="forcebalanced_manipulator" xmlns:xacro="http://ros.org/wiki/xacro">
+<robot name="forbal2" xmlns:xacro="http://ros.org/wiki/xacro">
+  <xacro:arg name="dummy" default="false"/>
   <xacro:include filename="$(find forbal_description)/urdf/forbal2.xacro" />
   <xacro:include filename="$(find forbal_description)/urdf/forbal2.ros2_control.xacro" />
@@ -7,5 +8,5 @@
     <origin xyz="0 0 0" rpy="0 0 0" />
   </xacro:forbal2>
-  <xacro:forbal_ros2_control name="forcebalanced_manipulator_ros2_control" dummy="false"/>
+  <xacro:forbal2_ros2_control name="forbal2" dummy="$(arg dummy)"/>
   <xacro:ringmass parent="link11" mass="0.02982881" density="8050.0" radius_inner="0.0032" radius_outer="0.02">
     <origin xyz="-0.2 0 0" rpy="0 0 0"/>

File: forbal_description/urdf/forbal5.ros2_control.xacro (robot description, xacro)
@@ -62,5 +62,5 @@
       <param name="Profile_Acceleration">0</param>
     </joint>
-    <joint name="jointem">
+    <joint name="joint3">
       <param name="id">3</param>
       <command_interface name="position"/>
@@ -77,5 +77,5 @@
       <param name="Profile_Acceleration">0</param>
     </joint>
-    <joint name="jointei">
+    <joint name="joint4">
       <param name="id">4</param>
       <command_interface name="position"/>

File: forbal_description/urdf/forbal5.xacro (robot description, xacro)
@@ -174,4 +174,11 @@
         <axis xyz="1 0 0"/>
     </joint>
+    <joint name="joint0" type="revolute">
+        <parent link="base"/>
+        <child link="mount"/>
+        <origin rpy="0.00000000 0.00000000 0.00000000" xyz="0.00000000 0.00000000 0.04600000"/>
+        <axis xyz="0.00000000 0.00000000 1.00000000"/>
+        <limit lower="-3.14159265" upper="3.14159265" effort="0" velocity="0"/>
+    </joint>
     <joint name="joint11" type="revolute">
         <parent link="mount"/>
@@ -181,10 +188,4 @@
         <limit lower="-3.14159265" upper="3.14159265" effort="0" velocity="0"/>
     </joint>
-    <joint name="joint11_cm" type="fixed">
-        <parent link="link11"/>
-        <child link="link11_cm"/>
-        <origin rpy="0.00000000 0.00000000 0.00000000" xyz="-0.20000000  0.00000000  0.00000000"/>
-        <axis xyz="1 0 0"/>
-    </joint>
     <joint name="joint12" type="revolute">
         <parent link="link11"/>
@@ -201,10 +202,4 @@
         <limit lower="-3.14159265" upper="3.14159265" effort="0" velocity="0"/>
     </joint>
-    <joint name="joint21_cm" type="fixed">
-        <parent link="link21"/>
-        <child link="link21_cm"/>
-        <origin rpy="0.00000000 0.00000000 0.00000000" xyz="-0.20000000  0.00000000  0.00000000"/>
-        <axis xyz="1 0 0"/>
-    </joint>
     <joint name="joint22" type="revolute">
         <parent link="link21"/>
@@ -214,21 +209,8 @@
         <limit lower="-3.14159265" upper="3.14159265" effort="0" velocity="0"/>
     </joint>
-    <joint name="joint22_cm" type="fixed">
-        <parent link="link22"/>
-        <child link="link22_cm"/>
-        <origin rpy="0.00000000 0.00000000 0.00000000" xyz="-0.20000000  0.00000000  0.00000000"/>
-        <axis xyz="1 0 0"/>
-    </joint>
-    <joint name="joint_ee_mkr" type="fixed">
-        <parent link="ee_imp"/>
-        <child link="ee_mkr"/>
-        <origin rpy="0.00000000 0.00000000 0.00000000" xyz="0.00750000 0.00000000 0.00000000"/>
-        <axis xyz="1 0 0"/>
-    </joint>
     <joint name="joint_lc1_l12" type="fixed">
         <parent link="link12"/>
         <child link="lc1"/>
         <origin rpy="0.00000000 0.00000000 0.00000000" xyz="0.20000000 0.04520000 0.00000000"/>
-        <axis xyz="1 0 0"/>
     </joint>
     <joint name="joint_lc_l22" type="fixed">
@@ -244,24 +226,22 @@
         <axis xyz="1 0 0"/>
     </joint>
-    <joint name="jointei" type="revolute">
+    <joint name="joint3" type="revolute">
+        <parent link="ee"/>
+        <child link="ee_motor"/>
+        <origin rpy="1.5707963268 0.0 0.0" xyz="0.025 -0.02100000 0.0"/>
+        <axis xyz="0.0 0.00000000 1.00000000"/>
+        <limit lower="-3.14159265" upper="3.14159265" effort="0" velocity="0"/>
+    </joint>
+    <joint name="joint4" type="revolute">
         <parent link="ee_motor"/>
         <child link="ee_imp"/>
-        <origin rpy="0.00000000 -1.57079633  0.00000000" xyz="0.01900000 -0.02400000 -0.01900000"/>
+        <origin rpy="0.0 -1.5707963268  0.00000000" xyz="0.019 -0.024 -0.019"/>
         <axis xyz="0.00000000 0.00000000 1.00000000"/>
         <limit lower="-3.14159265" upper="3.14159265" effort="0" velocity="0"/>
     </joint>
-    <joint name="jointem" type="revolute">
-        <parent link="ee"/>
-        <child link="ee_motor"/>
-        <origin rpy="1.57079633 -1.57079633  0.00000000" xyz="0.02500000 -0.02195000  0.00000000"/>
-        <axis xyz="0.00000000 0.00000000 1.00000000"/>
-        <limit lower="-3.14159265" upper="3.14159265" effort="0" velocity="0"/>
-    </joint>
-    <joint name="joint0" type="revolute">
-        <parent link="base"/>
-        <child link="mount"/>
-        <origin rpy="0.00000000 0.00000000 0.00000000" xyz="0.00000000 0.00000000 0.04600000"/>
-        <axis xyz="0.00000000 0.00000000 1.00000000"/>
-        <limit lower="-3.14159265" upper="3.14159265" effort="0" velocity="0"/>
+    <joint name="joint_ee_mkr" type="fixed">
+        <parent link="ee_imp"/>
+        <child link="ee_mkr"/>
+        <origin rpy="3.1415926536 0.0 -1.5707963268" xyz="0.0 -0.02 -0.01"/>
     </joint>
 </xacro:macro>

Commit message: All final changes to code and URDF to make forbal5 work + tuning

File: forbal_description/urdf/forbal2.ros2_control.xacro (robot description, xacro)
@@ -18,8 +18,8 @@
         <state_interface name="velocity"/>
         <state_interface name="effort"/>
-        <!-- <param name="Position_P_Gain">8000</param> -->
-        <!-- <param name="Position_D_Gain">12000</param> -->
-        <param name="Position_P_Gain">12500</param>
-        <param name="Position_D_Gain">16000</param>
+        <param name="Position_P_Gain">10000</param>
+        <param name="Position_D_Gain">12000</param>
+        <!-- <param name="Position_P_Gain">12500</param> -->
+        <!-- <param name="Position_D_Gain">16000</param> -->
         <param name="Position_I_Gain">0</param>
         <param name="Velocity_P_Gain">1920</param>
@@ -35,9 +35,9 @@
         <state_interface name="velocity"/>
         <state_interface name="effort"/>
-        <!-- <param name="Position_P_Gain">9000</param> -->
-        <!-- <param name="Position_D_Gain">13000</param> -->
+        <param name="Position_I_Gain">0</param>
         <param name="Position_P_Gain">15000</param>
-        <param name="Position_D_Gain">20000</param>
-        <param name="Position_I_Gain">0</param>
+        <param name="Position_D_Gain">18000</param>
+        <!-- <param name="Position_P_Gain">15000</param> -->
+        <!-- <param name="Position_D_Gain">20000</param> -->
         <param name="Velocity_P_Gain">1920</param>
         <param name="Velocity_I_Gain">0</param>

File: forbal_description/urdf/forbal5.ros2_control.xacro (robot description, xacro)
@@ -35,8 +35,8 @@
       <state_interface name="velocity"/>
       <state_interface name="effort"/>
-      <param name="Position_P_Gain">7000</param>
-      <param name="Position_D_Gain">14000</param>
-      <!-- <param name="Position_P_Gain">12500</param> -->
-      <!-- <param name="Position_D_Gain">16000</param> -->
+      <!-- <param name="Position_P_Gain">7000</param> -->
+      <!-- <param name="Position_D_Gain">14000</param> -->
+      <param name="Position_P_Gain">12500</param>
+      <param name="Position_D_Gain">16000</param>
       <param name="Position_I_Gain">0</param>
       <param name="Velocity_P_Gain">1920</param>
@@ -52,8 +52,8 @@
       <state_interface name="velocity"/>
       <state_interface name="effort"/>
-      <param name="Position_P_Gain">7000</param>
-      <param name="Position_D_Gain">14000</param>
-      <!-- <param name="Position_P_Gain">14000</param> -->
-      <!-- <param name="Position_D_Gain">16000</param> -->
+      <!-- <param name="Position_P_Gain">7000</param> -->
+      <!-- <param name="Position_D_Gain">14000</param> -->
+      <param name="Position_P_Gain">14000</param>
+      <param name="Position_D_Gain">16000</param>
       <param name="Position_I_Gain">0</param>
       <param name="Velocity_P_Gain">1920</param>

File: forbal_description/urdf/forbal5.xacro (robot description, xacro)
@@ -230,5 +230,5 @@
         <child link="ee_motor"/>
         <origin rpy="1.5707963268 -1.57079633 0.0" xyz="0.025 -0.01900000 0.0"/>
-        <axis xyz="0.0 0.00000000 1.00000000"/>
+        <axis xyz="0.0 0.00000000 -1.00000000"/>
         <limit lower="-2.0" upper="1.55" effort="0" velocity="0"/>
     </joint>
